File: KiCad/streamdeck/streamdeck.sch (KiCad schematic (older format))
At the start: 21 parts

Commit message: Last version
Parts:
- removed R? (x10): R, symbol Device:R
Connections:
- wire segments 78 -> 2
